File: schematics/experiment-tools-valve.sch (KiCad schematic (older format))
At the start: 4 parts, among them K1 Solenoid-Valve-12V, U1 Digispark_Attiny85, U2 TLP222A

Commit message: Fix solenoid valve connection
Connections:
- net +12V: now also K1.2, K1.8; no longer U2.4
- net GND: now also U2.3; no longer K1.1, K1.14
- new net: K1.1, K1.14, U2.4
Changed lines of the file:
@@
 	-1   0    0    -1
-$EndComp
-Wire Wire Line
-	7600 3700 7600 3750
-$Comp
-L power:GND #PWR?
-U 1 1 60A17D93
-P 7600 4350
-F 0 "#PWR?" H 7600 4100 50  0001 C CNN
-F 1 "GND" H 7605 4177 50  0000 C CNN
-F 2 "" H 7600 4350 50  0001 C CNN
-F 3 "" H 7600 4350 50  0001 C CNN
-	1    7600 4350
-	1    0    0    -1
 $EndComp
 $Comp
 L power:+12V #PWR?
 U 1 1 60A186C3
-P 6750 3900
-F 0 "#PWR?" H 6750 3750 50  0001 C CNN
-F 1 "+12V" H 6765 4073 50  0000 C CNN
-F 2 "" H 6750 3900 50  0001 C CNN
-F 3 "" H 6750 3900 50  0001 C CNN
-	1    6750 3900
+P 7600 3750
+F 0 "#PWR?" H 7600 3600 50  0001 C CNN
+F 1 "+12V" H 7615 3923 50  0000 C CNN
+F 2 "" H 7600 3750 50  0001 C CNN
+F 3 "" H 7600 3750 50  0001 C CNN
+	1    7600 3750
+	1    0    0    -1
+$EndComp
+$Comp
+L power:GND #PWR?
+U 1 1 609DEC4B
+P 6700 4150
+F 0 "#PWR?" H 6700 3900 50  0001 C CNN
+F 1 "GND" H 6705 3977 50  0000 C CNN
+F 2 "" H 6700 4150 50  0001 C CNN
+F 3 "" H 6700 4150 50  0001 C CNN
+	1    6700 4150
 	1    0    0    -1
 $EndComp
 Wire Wire Line
-	6700 3950 6750 3950
+	7600 4350 7050 4350
 Wire Wire Line
-	6750 3950 6750 3900
+	7050 4350 7050 3950
 Wire Wire Line
-	6700 4150 7100 4150
-Wire Wire Line
-	7100 4150 7100 3700
-Wire Wire Line
-	7100 3700 7600 3700
+	6700 3950 7050 3950
 $EndSCHEMATC
